File: MM8I Mk2/MM8I Mk2.brd (EAGLE design)
At the start: 160 x 100 mm, 14 parts, among them U1 CY14B104M, U2 SN74LVC16T245DGVR

Commit message: Progress on MM8I Mk2
Parts:
- removed C2, C3: (no value), rcl:C0805
- added U3: SN74LVCH16374ADGGR, MM24I:DGG48
- added U4: SN74AHCT16373DGGR, MM24I:DGG48
- U2: value SN74LVC16T245DGVR -> SN74LVCH16374ADGGR; device MM24I:DGV48 -> MM24I:DGG48
- moved U2 43.1 mm to (-67.3, -127.0)
Connections:
- removed net N$18: U2.2
- removed net N$19: U2.3
- removed net N$20: U2.5
- removed net N$21: U2.6
- removed net N$22: U2.8
- removed net N$23: U2.9
- removed net N$24: U2.11
- removed net N$25: U2.12
- removed net N$26: U2.13
- removed net N$27: U2.14
- removed net N$28: U2.16
- removed net N$29: U2.17
- new net N$32: U1.3, U3.13
- new net N$33: U1.4, U3.14
- new net N$34: U1.6, U3.17
- new net N$36: U1.7, U3.19
- new net N$37: U1.20, U3.20
- new net N$38: U1.21, U3.22
- new net N$39: U1.22, U3.23
- new net N$40: U1.24, U3.3
- new net N$41: U1.31, U3.5
- new net N$42: U1.32, U3.6
- new net N$43: U1.33, U3.8
- new net N$44: U1.34, U3.9
- new net N$45: U1.35, U3.11
- net !WE: no longer U2.1, U2.24
- net +5V: now also U4.18, U4.31, U4.42, U4.7; no longer C3.2
- net GND: now also R1.1, R2.1, R3.1, R4.1, U1.47, U1.48, U1.50, U1.51, U1.52, U1.8, U2.1, U2.24, U3.1, U3.10, U3.15, U3.21, U3.24, U3.26, U3.28, U3.34, U3.39, U3.4, U3.45, U4.1, U4.10, U4.15, U4.21, U4.24, U4.26, U4.27, U4.28, U4.29, U4.30, U4.34, U4.39, U4.4, U4.45; no longer R1.2, R2.2, R3.2, R4.2, U2.19, U2.20, U2.22, U2.23, U2.25, U2.48
- net MCS-MEM-00-H: now also U4.2
- net MCS-MEM-01-H: now also U4.3
- net MCS-MEM-02-H: now also U4.5
- net MCS-MEM-03-H: now also U4.6
- net MCS-MEM-04-H: now also U4.8
- net MCS-MEM-05-H: now also U4.9
- net MCS-MEM-06-H: now also U4.11
- net MCS-MEM-07-H: now also U4.12
- net MCS-MEM-08-H: now also U4.13
- net MCS-MEM-09-H: now also U4.14
- net MCS-MEM-10-H: now also U4.16
- net MCS-MEM-11-H: now also U4.17
- net MXB-BMA-00-H: now also U3.47
- net MXB-BMA-01-H: now also U3.46
- net MXB-BMA-02-H: now also U3.44
- net MXB-BMA-03-H: now also U3.43
- net MXB-BMA-04-H: now also U3.41
- net MXB-BMA-05-H: now also U3.40
- net MXB-BMA-06-H: now also U3.38
- net MXB-BMA-07-H: now also U3.37
- net MXB-BMA-08-H: now also U3.36
- net MXB-BMA-09-H: now also U3.35
- net MXB-BMA-10-H: now also U3.33
- net MXB-BMA-11-H: now also U3.32
- net MXB-MCBMB-00-H: now also U2.47
- net MXB-MCBMB-01-H: now also U2.46
- net MXB-MCBMB-02-H: now also U2.44
- net MXB-MCBMB-03-H: now also U2.43
- net MXB-MCBMB-04-H: now also U2.41
- net MXB-MCBMB-05-H: now also U2.40
- net MXB-MCBMB-06-H: now also U2.38
- net MXB-MCBMB-07-H: now also U2.37
- net MXB-MCBMB-08-H: now also U2.36
- net MXB-MCBMB-09-H: now also U2.35
- net MXB-MCBMB-10-H: now also U2.33
- net MXB-MCBMB-11-H: now also U2.32
- net MXF-EA-00-H: now also U3.30
- net MXF-EA-01-H: now also U3.29
- net MXF-EA-02-H: now also U3.27
- net N$10: now also R2.2, U1.45; no longer R4.1, U1.46
- net N$11: now also U2.22, U4.38; no longer U2.38
- net N$12: now also R3.2, U1.44; no longer R1.1, U1.43
- net N$13: now also U2.23, U4.37; no longer U2.37
- net N$14: now also U2.2, U4.36; no longer U2.36
- net N$15: now also U2.3, U4.35; no longer U2.35
- net N$16: now also U2.5, U4.33; no longer U2.33
- net N$17: now also U2.6, U4.32; no longer U2.32
- net N$2: now also U2.13, U4.47; no longer U2.47
- net N$3: now also U2.14, U4.46; no longer U2.46
- net N$30: now also U1.23, U3.2; no longer C3.1, U2.18, U2.7
- net N$31: now also U1.5, U3.16; no longer C2.1, U2.31, U2.42
- net N$4: now also U2.16, U4.44; no longer U2.44
- net N$5: now also U2.17, U4.43; no longer U2.43
- net N$6: now also U2.19, U4.41; no longer U2.41
- net N$7: now also U2.20, U4.40; no longer U2.40
- net N$8: now also R4.2, U1.43; no longer R2.1, U1.44
- net N$9: now also R1.2, U1.46; no longer R3.1, U1.45
- net VCC: now also U2.18, U2.31, U2.42, U2.7, U3.18, U3.31, U3.42, U3.7; no longer C2.2

Commit message: First board layout revision
Parts:
- removed N20, N21, N22, N23, N24: FH21-18S-1DSA, con-hirose:FH21-18S-1DSA
- added C2: 0.47UF, MM24I:CC0603N
- added C3: 47UF, MM24I:NOJC
- added DL1, DL2: 50-500 ns, MM24I:21-0066J_14
- added IC1: SN74LVC2G17DBVR, MM24I:DBV6
- added IC2: SN74LVC14APWR, MM24I:PW14
- added VR1: LM3940IMP-3.3, MM24I:MP04A
- added X1, X2, X3, X4, X5: FH21-18S-1DSA, con-hirose:FH21-18S-1DSA
- U1: value CY14B104M -> SN74LVCH16374ADGGR; device MM24I:TSOPII-54 -> MM24I:DGG48
- U3: value SN74LVCH16374ADGGR -> CY14B104M; device MM24I:DGG48 -> MM24I:TSOPII-54
- moved U3 206.1 mm to (71.9, 15.0), turned to 270 degrees
- moved U2 192.4 mm to (34.9, 36.0)
- moved U4 165.9 mm to (34.9, 11.0)
- moved R4 134.3 mm to (74.3, 40.8)
- moved R3 129.0 mm to (74.3, 37.1)
- moved U1 125.0 mm to (34.9, 62.0)
- moved R2 124.1 mm to (74.3, 33.4)
- moved R1 119.6 mm to (74.3, 29.7)
- moved C1 103.8 mm to (65.5, 31.0), turned to 180 degrees
Connections:
- removed net !WE: U1.19
- new net !MEM-DONE: DL2.8, IC2.3
- new net !STROBE: DL1.8, IC2.1
- new net !WRITE-ENABLE: IC2.6, U3.19
- new net LATCH-MA: DL1.4, U2.25, U2.48
- new net LATCH-MB: DL2.5, U1.25, U1.48
- new net LATCH-MEM: DL1.9, U4.25, U4.48
- new net START-MEMORY: DL1.1, IC1.6
- new net TIMING-PULSE-3: DL2.1, IC1.4
- new net WRITE-ENABLE: DL2.10, IC2.5, U3.49
- net +5V: now also C2.1, VR1.1
- net GND: now also C2.2, C3.2, DL1.7, DL2.7, IC1.2, IC2.11, IC2.13, IC2.7, IC2.9, U1.1, U1.10, U1.15, U1.21, U1.24, U1.26, U1.27, U1.30, U1.34, U1.39, U1.4, U1.45, U3.14, U3.42, U3.47, U3.48, U3.50, U3.51, U3.52, U3.8, VR1.2, VR1.4, X1.10, X1.12, X1.14, X1.17, X1.3, X1.6, X1.8, X2.10, X2.12, X2.14, X2.17, X2.3, X2.6, X2.8, X3.10, X3.12, X3.14, X3.17, X3.3, X3.6, X3.8, X4.10, X4.12, X4.14, X4.17, X4.3, X4.6, X4.8, X5.10, X5.12, X5.14, X5.17, X5.3, X5.6, X5.8; no longer N20.10, N20.12, N20.14, N20.17, N20.3, N20.6, N20.8, N21.10, N21.12, N21.14, N21.17, N21.3, N21.6, N21.8, N22.10, N22.12, N22.14, N22.17, N22.3, N22.6, N22.8, N23.10, N23.12, N23.14, N23.17, N23.3, N23.6, N23.8, N24.10, N24.12, N24.14, N24.17, N24.3, N24.6, N24.8, U1.14, U1.42, U1.47, U1.48, U1.50, U1.51, U1.52, U1.8, U2.27, U2.29, U2.30, U3.1, U3.10, U3.15, U3.21, U3.24, U3.26, U3.28, U3.34, U3.39, U3.4, U3.45
- net MCS-MEM-00-H: now also X4.5; no longer N23.5
- net MCS-MEM-01-H: now also X4.7; no longer N23.7
- net MCS-MEM-02-H: now also X4.9; no longer N23.9
- net MCS-MEM-03-H: now also X4.11; no longer N23.11
- net MCS-MEM-04-H: now also X4.13; no longer N23.13
- net MCS-MEM-05-H: now also X4.15; no longer N23.15
- net MCS-MEM-06-H: now also X4.16; no longer N23.16
- net MCS-MEM-07-H: now also X4.18; no longer N23.18
- net MCS-MEM-08-H: now also X5.4; no longer N24.4
- net MCS-MEM-09-H: now also X5.5; no longer N24.5
- net MCS-MEM-10-H: now also X5.7; no longer N24.7
- net MCS-MEM-11-H: now also X5.9; no longer N24.9
- net MCT-MEM-DONE-L: now also IC2.4, X5.15; no longer N24.15
- net MCT-STROBE-L: now also IC2.2, X5.13; no longer N24.13
- net MXB-BMA-00-H: now also U2.47, X1.9; no longer N20.9, U3.47
- net MXB-BMA-01-H: now also U2.46, X1.11; no longer N20.11, U3.46
- net MXB-BMA-02-H: now also U2.44, X1.13; no longer N20.13, U3.44
- net MXB-BMA-03-H: now also U2.43, X1.15; no longer N20.15, U3.43
- net MXB-BMA-04-H: now also U2.41, X1.16; no longer N20.16, U3.41
- net MXB-BMA-05-H: now also U2.40, X1.18; no longer N20.18, U3.40
- net MXB-BMA-06-H: now also U2.38, X2.4; no longer N21.4, U3.38
- net MXB-BMA-07-H: now also U2.37, X2.5; no longer N21.5, U3.37
- net MXB-BMA-08-H: now also U2.36, X2.7; no longer N21.7, U3.36
- net MXB-BMA-09-H: now also U2.35, X2.9; no longer N21.9, U3.35
- net MXB-BMA-10-H: now also U2.33, X2.11; no longer N21.11, U3.33
- net MXB-BMA-11-H: now also U2.32, X2.13; no longer N21.13, U3.32
- net MXB-MCBMB-00-H: now also U1.47, X2.15; no longer N21.15, U2.47
- net MXB-MCBMB-01-H: now also U1.46, X2.16; no longer N21.16, U2.46
- net MXB-MCBMB-02-H: now also U1.44, X2.18; no longer N21.18, U2.44
- net MXB-MCBMB-03-H: now also U1.43, X1.4; no longer N20.4, U2.43
- net MXB-MCBMB-04-H: now also U1.41, X1.5; no longer N20.5, U2.41
- net MXB-MCBMB-05-H: now also U1.40, X1.7; no longer N20.7, U2.40
- net MXB-MCBMB-06-H: now also U1.38, X3.9; no longer N22.9, U2.38
- net MXB-MCBMB-07-H: now also U1.37, X3.11; no longer N22.11, U2.37
- net MXB-MCBMB-08-H: now also U1.36, X3.13; no longer N22.13, U2.36
- net MXB-MCBMB-09-H: now also U1.35, X3.15; no longer N22.15, U2.35
- net MXB-MCBMB-10-H: now also U1.33, X3.16; no longer N22.16, U2.33
- net MXB-MCBMB-11-H: now also U1.32, X3.18; no longer N22.18, U2.32
- net MXB-MEM-TP3-H: now also IC1.3, X5.18; no longer N24.18
- net MXB-START-MEMORY-H: now also IC1.1, X5.11; no longer N24.11
- net MXF-EA-00-H: now also U2.30, X3.4; no longer N22.4, U3.30
- net MXF-EA-01-H: now also U2.29, X3.5; no longer N22.5, U3.29
- net MXF-EA-02-H: now also U2.27, X3.7; no longer N22.7, U3.27
- net N$1: now also U3.36; no longer U1.36
- net N$10: now also U3.45; no longer U1.45
- net N$11: now also U1.22, U3.17; no longer U1.17, U2.22
- net N$12: now also U3.44; no longer U1.44
- net N$13: now also U1.23, U3.18; no longer U1.18, U2.23
- net N$14: now also U1.2, U3.37; no longer U1.37, U2.2
- net N$15: now also U1.3, U3.38; no longer U1.38, U2.3
- net N$16: now also U1.5, U3.39; no longer U1.39, U2.5
- net N$17: now also U1.6, U3.40; no longer U1.40, U2.6
- net N$2: now also U1.13, U3.9; no longer U1.9, U2.13
- net N$3: now also U1.14, U3.10; no longer U1.10, U2.14
- net N$30: now also U2.2, U3.23; no longer U1.23, U3.2
- net N$31: now also U2.16, U3.5; no longer U1.5, U3.16
- net N$32: now also U2.13, U3.3; no longer U1.3, U3.13
- net N$33: now also U2.14, U3.4; no longer U1.4, U3.14
- net N$34: now also U2.17, U3.6; no longer U1.6, U3.17
- net N$36: now also U2.19, U3.7; no longer U1.7, U3.19
- net N$37: now also U2.20; no longer U1.20
- net N$38: now also U2.22, U3.21; no longer U1.21, U3.22
- net N$39: now also U2.23, U3.22; no longer U1.22, U3.23
- net N$4: now also U1.16, U3.11; no longer U1.11, U2.16
- net N$40: now also U2.3, U3.24; no longer U1.24, U3.3
- net N$41: now also U2.5, U3.31; no longer U1.31, U3.5
- net N$42: now also U2.6, U3.32; no longer U1.32, U3.6
- net N$43: now also U2.8, U3.33; no longer U1.33, U3.8
- net N$44: now also U2.9, U3.34; no longer U1.34, U3.9
- net N$45: now also U2.11, U3.35; no longer U1.35, U3.11
- net N$5: now also U1.17, U3.12; no longer U1.12, U2.17
- net N$6: now also U1.19, U3.15; no longer U1.15, U2.19
- net N$7: now also U1.20, U3.16; no longer U1.16, U2.20
- net N$8: now also U3.43; no longer U1.43
- net N$9: now also U3.46; no longer U1.46
- net VCC: now also C3.1, DL1.14, DL2.14, IC1.5, IC2.14, U1.18, U1.31, U1.42, U1.7, U3.13, U3.41, VR1.3; no longer U1.13, U1.41, U3.18, U3.31, U3.42, U3.7
Routing:
- net N$16: track 0.00 -> 143.7 mm, vias 0 -> 3
- net N$14: track 0.00 -> 118.3 mm, vias 0 -> 5
- net N$15: track 0.00 -> 117.3 mm, vias 0 -> 4
- net N$17: track 0.00 -> 106.8 mm, vias 0 -> 4
- net GND: track 0.00 -> 102.5 mm, vias 0 -> 48
- net N$6: track 0.00 -> 99.9 mm, vias 0 -> 4
- net N$41: track 0.00 -> 96.4 mm, vias 0 -> 2
- net N$44: track 0.00 -> 96.1 mm, vias 0 -> 2
- net +5V: track 0.00 -> 95.4 mm, vias 0 -> 4
- net N$45: track 0.00 -> 94.2 mm, vias 0 -> 2
- net N$4: track 0.00 -> 94.0 mm, vias 0 -> 6
- net N$2: track 0.00 -> 86.9 mm, vias 0 -> 4
- net N$5: track 0.00 -> 85.9 mm, vias 0 -> 2
- net N$3: track 0.00 -> 84.6 mm, vias 0 -> 4
- net N$40: track 0.00 -> 84.5 mm, vias 0 -> 2
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- added copper zone on layer 2, net GND
- added copper zone on layer 15, net VCC
Other:
- board size 160 x 100 mm -> 80.4 x 77 mm
