File: MM8I Mk2/MM8I Mk2.sch (EAGLE design)
At the start: 14 parts, among them U1 CY14B104M, U2 SN74LVCH16374ADGGR, U3 SN74LVCH16374ADGGR, U4 SN74AHCT16373DGGR

Commit message: First board layout revision
Parts:
- removed N20, N21, N22, N23, N24: FH21-18S-1DSA, con-hirose:FH21-18S-1DSA
- added C2: 0.47UF, MM24I:C0603C474K8PACTU
- added C3: 47UF, MM24I:NOJC476M010RWJ
- added DL1, DL2: 50-500 ns, MM24I:DS1110LE-500+
- added IC1: SN74LVC2G17DBVR, MM24I:SN74LVC2G17DBVR
- added IC2: SN74LVC14APWR, MM24I:SN74LVC14APWR
- added VR1: LM3940IMP-3.3, MM24I:LM3940IMP-3.3
- added X1, X2, X3, X4, X5: FH21-18S-1DSA, con-hirose:FH21-18S-1DSA
- U1: value CY14B104M -> SN74LVCH16374ADGGR; device MM24I:CY14B104M -> MM24I:SN74LVCH16374ADGGR
- U3: value SN74LVCH16374ADGGR -> CY14B104M; device MM24I:SN74LVCH16374ADGGR -> MM24I:CY14B104M
Connections:
- removed net !WE: U1.!WE
- new net !MEM-DONE: DL2.TAP10, IC2.2A
- new net !STROBE: DL1.TAP10, IC2.1A
- new net !WRITE-ENABLE: IC2.3Y, U3.!WE
- new net LATCH-MA: DL1.TAP4, U2A.1CLK, U2A.2CLK
- new net LATCH-MB: DL2.TAP6, U1A.1CLK, U1A.2CLK
- new net LATCH-MEM: DL1.TAP9, U4A.1LE, U4A.2LE
- new net START-MEMORY: DL1.IN, IC1.1Y
- new net TIMING-PULSE-3: DL2.IN, IC1.2Y
- new net WRITE-ENABLE: DL2.TAP7, IC2.3A, U3.!OE
- net +5V: now also C2.1, VR1.IN
- net GND: now also C2.2, C3.C2, DL1.GND, DL2.GND, IC1.GND, IC2.4A, IC2.5A, IC2.6A, IC2.GND, U1A.!1OE, U1A.!2OE, U1A.2D5, U1A.2D6, U1A.2D7, U1A.2D8, U1B.GND@10, U1B.GND@15, U1B.GND@21, U1B.GND@28, U1B.GND@34, U1B.GND@39, U1B.GND@4, U1B.GND@45, U3.!BHE, U3.!BLE, U3.!CE, U3.A15, U3.A16, U3.A17, U3.VSS@14, U3.VSS@42, VR1.GND@2, VR1.GND@4, X1.10, X1.12, X1.14, X1.17, X1.3, X1.6, X1.8, X2.10, X2.12, X2.14, X2.17, X2.3, X2.6, X2.8, X3.10, X3.12, X3.14, X3.17, X3.3, X3.6, X3.8, X4.10, X4.12, X4.14, X4.17, X4.3, X4.6, X4.8, X5.10, X5.12, X5.14, X5.17, X5.3, X5.6, X5.8; no longer N20.10, N20.12, N20.14, N20.17, N20.3, N20.6, N20.8, N21.10, N21.12, N21.14, N21.17, N21.3, N21.6, N21.8, N22.10, N22.12, N22.14, N22.17, N22.3, N22.6, N22.8, N23.10, N23.12, N23.14, N23.17, N23.3, N23.6, N23.8, N24.10, N24.12, N24.14, N24.17, N24.3, N24.6, N24.8, U1.!BHE, U1.!BLE, U1.!CE, U1.A15, U1.A16, U1.A17, U1.VRTCBAT, U1.VRTCCAP, U1.VSS@14, U1.VSS@42, U2A.2D5, U2A.2D6, U2A.2D7, U3A.!1OE, U3A.!2OE, U3A.2D8, U3B.GND@10, U3B.GND@15, U3B.GND@21, U3B.GND@28, U3B.GND@34, U3B.GND@39, U3B.GND@4, U3B.GND@45
- net MCS-MEM-00-H: now also X4.5; no longer N23.5
- net MCS-MEM-01-H: now also X4.7; no longer N23.7
- net MCS-MEM-02-H: now also X4.9; no longer N23.9
- net MCS-MEM-03-H: now also X4.11; no longer N23.11
- net MCS-MEM-04-H: now also X4.13; no longer N23.13
- net MCS-MEM-05-H: now also X4.15; no longer N23.15
- net MCS-MEM-06-H: now also X4.16; no longer N23.16
- net MCS-MEM-07-H: now also X4.18; no longer N23.18
- net MCS-MEM-08-H: now also X5.4; no longer N24.4
- net MCS-MEM-09-H: now also X5.5; no longer N24.5
- net MCS-MEM-10-H: now also X5.7; no longer N24.7
- net MCS-MEM-11-H: now also X5.9; no longer N24.9
- net MCT-MEM-DONE-L: now also IC2.2Y, X5.15; no longer N24.15
- net MCT-STROBE-L: now also IC2.1Y, X5.13; no longer N24.13
- net MXB-BMA-00-H: now also U2A.1D1, X1.9; no longer N20.9, U3A.1D1
- net MXB-BMA-01-H: now also U2A.1D2, X1.11; no longer N20.11, U3A.1D2
- net MXB-BMA-02-H: now also U2A.1D3, X1.13; no longer N20.13, U3A.1D3
- net MXB-BMA-03-H: now also U2A.1D4, X1.15; no longer N20.15, U3A.1D4
- net MXB-BMA-04-H: now also U2A.1D5, X1.16; no longer N20.16, U3A.1D5
- net MXB-BMA-05-H: now also U2A.1D6, X1.18; no longer N20.18, U3A.1D6
- net MXB-BMA-06-H: now also U2A.1D7, X2.4; no longer N21.4, U3A.1D7
- net MXB-BMA-07-H: now also U2A.1D8, X2.5; no longer N21.5, U3A.1D8
- net MXB-BMA-08-H: now also U2A.2D1, X2.7; no longer N21.7, U3A.2D1
- net MXB-BMA-09-H: now also U2A.2D2, X2.9; no longer N21.9, U3A.2D2
- net MXB-BMA-10-H: now also U2A.2D3, X2.11; no longer N21.11, U3A.2D3
- net MXB-BMA-11-H: now also U2A.2D4, X2.13; no longer N21.13, U3A.2D4
- net MXB-MCBMB-00-H: now also U1A.1D1, X2.15; no longer N21.15, U2A.1D1
- net MXB-MCBMB-01-H: now also U1A.1D2, X2.16; no longer N21.16, U2A.1D2
- net MXB-MCBMB-02-H: now also U1A.1D3, X2.18; no longer N21.18, U2A.1D3
- net MXB-MCBMB-03-H: now also U1A.1D4, X1.4; no longer N20.4, U2A.1D4
- net MXB-MCBMB-04-H: now also U1A.1D5, X1.5; no longer N20.5, U2A.1D5
- net MXB-MCBMB-05-H: now also U1A.1D6, X1.7; no longer N20.7, U2A.1D6
- net MXB-MCBMB-06-H: now also U1A.1D7, X3.9; no longer N22.9, U2A.1D7
- net MXB-MCBMB-07-H: now also U1A.1D8, X3.11; no longer N22.11, U2A.1D8
- net MXB-MCBMB-08-H: now also U1A.2D1, X3.13; no longer N22.13, U2A.2D1
- net MXB-MCBMB-09-H: now also U1A.2D2, X3.15; no longer N22.15, U2A.2D2
- net MXB-MCBMB-10-H: now also U1A.2D3, X3.16; no longer N22.16, U2A.2D3
- net MXB-MCBMB-11-H: now also U1A.2D4, X3.18; no longer N22.18, U2A.2D4
- net MXB-MEM-TP3-H: now also IC1.2A, X5.18; no longer N24.18
- net MXB-START-MEMORY-H: now also IC1.1A, X5.11; no longer N24.11
- net MXF-EA-00-H: now also U2A.2D5, X3.4; no longer N22.4, U3A.2D5
- net MXF-EA-01-H: now also U2A.2D6, X3.5; no longer N22.5, U3A.2D6
- net MXF-EA-02-H: now also U2A.2D7, X3.7; no longer N22.7, U3A.2D7
- net N$1: now also U3.VCAP; no longer U1.VCAP
- net N$10: now also U3.DQ14; no longer U1.DQ14
- net N$11: now also U1A.1Q7, U3.DQ6; no longer U1.DQ6, U2A.1Q7
- net N$12: now also U3.DQ13; no longer U1.DQ13
- net N$13: now also U1A.1Q8, U3.DQ7; no longer U1.DQ7, U2A.1Q8
- net N$14: now also U1A.2Q1, U3.DQ8; no longer U1.DQ8, U2A.2Q1
- net N$15: now also U1A.2Q2, U3.DQ9; no longer U1.DQ9, U2A.2Q2
- net N$16: now also U1A.2Q3, U3.DQ10; no longer U1.DQ10, U2A.2Q3
- net N$17: now also U1A.2Q4, U3.DQ11; no longer U1.DQ11, U2A.2Q4
- net N$2: now also U1A.1Q1, U3.DQ0; no longer U1.DQ0, U2A.1Q1
- net N$3: now also U1A.1Q2, U3.DQ1; no longer U1.DQ1, U2A.1Q2
- net N$30: now also U2A.2Q1, U3.A8; no longer U1.A8, U3A.2Q1
- net N$31: now also U2A.1Q3, U3.A2; no longer U1.A2, U3A.1Q3
- net N$32: now also U2A.1Q1, U3.A0; no longer U1.A0, U3A.1Q1
- net N$33: now also U2A.1Q2, U3.A1; no longer U1.A1, U3A.1Q2
- net N$34: now also U2A.1Q4, U3.A3; no longer U1.A3, U3A.1Q4
- net N$36: now also U2A.1Q5, U3.A4; no longer U1.A4, U3A.1Q5
- net N$37: now also U2A.1Q6, U3.A5; no longer U1.A5, U3A.1Q6
- net N$38: now also U2A.1Q7, U3.A6; no longer U1.A6, U3A.1Q7
- net N$39: now also U2A.1Q8, U3.A7; no longer U1.A7, U3A.1Q8
- net N$4: now also U1A.1Q3, U3.DQ2; no longer U1.DQ2, U2A.1Q3
- net N$40: now also U2A.2Q2, U3.A9; no longer U1.A9, U3A.2Q2
- net N$41: now also U2A.2Q3, U3.A10; no longer U1.A10, U3A.2Q3
- net N$42: now also U2A.2Q4, U3.A11; no longer U1.A11, U3A.2Q4
- net N$43: now also U2A.2Q5, U3.A12; no longer U1.A12, U3A.2Q5
- net N$44: now also U2A.2Q6, U3.A13; no longer U1.A13, U3A.2Q6
- net N$45: now also U2A.2Q7, U3.A14; no longer U1.A14, U3A.2Q7
- net N$5: now also U1A.1Q4, U3.DQ3; no longer U1.DQ3, U2A.1Q4
- net N$6: now also U1A.1Q5, U3.DQ4; no longer U1.DQ4, U2A.1Q5
- net N$7: now also U1A.1Q6, U3.DQ5; no longer U1.DQ5, U2A.1Q6
- net N$8: now also U3.DQ12; no longer U1.DQ12
- net N$9: now also U3.DQ15; no longer U1.DQ15
- net VCC: now also C3.C1, DL1.VCC, DL2.VCC, IC1.VCC, IC2.VCC, U1B.VCC@18, U1B.VCC@31, U1B.VCC@42, U1B.VCC@7, U3.VCC@13, U3.VCC@41, VR1.OUT; no longer U1.VCC@13, U1.VCC@41, U3B.VCC@18, U3B.VCC@31, U3B.VCC@42, U3B.VCC@7
Other:
- note added: "Inverter"
- note added: "Schmitt Trigger Buffer"
- note removed: "SN74AHCT16373DGGR - 5v part, TTL input levels"
